Commit message: squashing commits

File: my_robot/urdf/my_robot.xacro (robot description, xacro)
@@ -204,5 +204,5 @@
   </link>
   <joint type="fixed" name="hokuyo_joint">
-    <origin xyz=".15 0 .05" rpy="0 0 0"/>
+    <origin xyz=".2 0 .25" rpy="0 0 0"/>
     <child link="hokuyo"/>
     <parent link="chassis"/>

Commit message: amcl tuning, robot description changes

File: my_robot/urdf/my_robot.xacro (robot description, xacro)
@@ -4,5 +4,5 @@
   <link name="robot_footprint"></link>
   <joint name="robot_footprint_joint" type="fixed">
-    <origin xyz="0 0 0" rpy="0 0 0" />
+    <origin xyz="0 0 .1" rpy="0 0 0" />
     <parent link="robot_footprint"/>
     <child link="chassis" />
@@ -186,5 +186,5 @@
   <link name="hokuyo">
     <collision>
-      <origin xyz="0 0 0" rpy="0 0 0"/>
+      <origin xyz="0 0 .25" rpy="0 0 0"/>
       <geometry>
 	<box size="0.1 0.1 0.1"/>
@@ -192,5 +192,5 @@
     </collision>
     <visual>
-      <origin xyz="0 0 0" rpy="0 0 0"/>
+      <origin xyz="0 0 .25" rpy="0 0 0"/>
       <geometry>
         <mesh filename="package://my_robot/meshes/hokuyo.dae"/>

Commit message: made new map, changed urdf to reflect chassis/robot footprint offset, amcl tuning

File: my_robot/urdf/my_robot.xacro (robot description, xacro)
@@ -4,5 +4,5 @@
   <link name="robot_footprint"></link>
   <joint name="robot_footprint_joint" type="fixed">
-    <origin xyz="0 0 .1" rpy="0 0 0" />
+    <origin xyz="0 0 .2" rpy="0 0 0" />
     <parent link="robot_footprint"/>
     <child link="chassis" />

Commit message: pre submit push

File: my_robot/urdf/my_robot.xacro (robot description, xacro)
@@ -186,11 +186,11 @@
   <link name="hokuyo">
     <collision>
-      <origin xyz="0 0 .25" rpy="0 0 0"/>
-      <geometry>
-	<box size="0.1 0.1 0.1"/>
+      <origin xyz="0 0 0" rpy="0 0 0"/>
+      <geometry>
+	<box size="0.1 0.1 0.0"/>
       </geometry>
     </collision>
     <visual>
-      <origin xyz="0 0 .25" rpy="0 0 0"/>
+      <origin xyz="0 0 0" rpy="0 0 0"/>
       <geometry>
         <mesh filename="package://my_robot/meshes/hokuyo.dae"/>
@@ -204,5 +204,5 @@
   </link>
   <joint type="fixed" name="hokuyo_joint">
-    <origin xyz=".2 0 .25" rpy="0 0 0"/>
+    <origin xyz=".2 0 0" rpy="0 0 0"/>
     <child link="hokuyo"/>
     <parent link="chassis"/>

Commit message: fixed urdf spawn crash issue - removed my_robot content from world file

File: my_robot/urdf/my_robot.xacro (robot description, xacro)
@@ -188,5 +188,5 @@
       <origin xyz="0 0 0" rpy="0 0 0"/>
       <geometry>
-	<box size="0.1 0.1 0.0"/>
+	<box size="0.1 0.1 0.1"/>
       </geometry>
     </collision>

Commit message: removed files from localization, made changes to robot urdf

File: my_robot/urdf/my_robot.xacro (robot description, xacro)
@@ -183,4 +183,11 @@
     <axis xyz="0 1 0" rpy="0 0 0"/>
   </joint>
+  <joint name="camera_optical_joint" type="fixed">
+    <origin xyz="0 0 0" rpy="-1.5707 0 -1.5707"/>
+    <parent link="camera"/>
+    <child link="camera_link_optical"/>
+  </joint>
+  <link name="camera_link_optical">
+  </link>
   <!-- Hokuyo Laser -->
   <link name="hokuyo">
